File: adapter/adapter.kicad_pcb (KiCad board)
At the start: 2 copper layers, 93.6 x 71.8 mm, 44 parts, among them J10 Ribbon, J11 Ribbon, J12 Ribbon, J13 serial, J14 serial, J3 battery charge, J6 battery charge, J7 trackball, J8 trackball, J9 Ribbon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

Commit message: fixed col6 and gnd fills
Routing:
- net col6_l: track 0.00 -> 26.6 mm
- net GND: track 94.0 -> 113.4 mm
Changed lines of the file:
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@@
   (segment (start 134.764684 108.364999) (end 134.764684 96.735316) (width 0.25) (layer "F.Cu") (net 13))
   (segment (start 132.689684 110.439999) (end 134.764684 108.364999) (width 0.25) (layer "F.Cu") (net 13))
+  (segment (start 132.9 96.4) (end 132.9 100.6) (width 0.25) (layer "F.Cu") (net 14))
+  (segment (start 132.9 100.6) (end 131.2 100.6) (width 0.25) (layer "F.Cu") (net 14))
+  (segment (start 131.1 94.6) (end 132.9 96.4) (width 0.25) (layer "F.Cu") (net 14))
+  (segment (start 125.94 94.6) (end 131.1 94.6) (width 0.25) (layer "F.Cu") (net 14))
+  (segment (start 131.225 111.515315) (end 132.689684 112.979999) (width 0.25) (layer "F.Cu") (net 14))
+  (segment (start 131.225 100.625) (end 131.225 111.515315) (width 0.25) (layer "F.Cu") (net 14))
+  (segment (start 131.2 100.6) (end 131.225 100.625) (width 0.25) (layer "F.Cu") (net 14))
   (segment (start 135.664684 112.544999) (end 135.664684 102.426716) (width 0.25) (layer "F.Cu") (net 15))
   (segment (start 135.664684 102.426716) (end 140.9514 97.14) (width 0.25) (layer "F.Cu") (net 15))
@@
   (segment (start 177.847199 115.499999) (end 181 112.347198) (width 0.25) (layer "F.Cu") (net 26))
   (segment (start 181 112.347198) (end 181 101.1314) (width 0.25) (layer "F.Cu") (net 26))
+  (segment (start 123.95 69.75) (end 125.94 71.74) (width 0.25) (layer "F.Cu") (net 27))
+  (segment (start 118.5 69.75) (end 123.95 69.75) (width 0.25) (layer "F.Cu") (net 27))
   (via (at 182.5 83) (size 0.8) (drill 0.4) (layers "F.Cu" "B.Cu") (free) (net 27))
   (via (at 133.5 85.25) (size 0.8) (drill 0.4) (layers "F.Cu" "B.Cu") (free) (net 27))
@@
   (segment (start 193.05 90.81) (end 193.05 98.086396) (width 0.25) (layer "B.Cu") (net 27))
   (segment (start 190.8 98.7) (end 190.8 113.15) (width 0.25) (layer "B.Cu") (net 27))
+  (segment (start 193.3 70.95) (end 188.55 70.95) (width 0.25) (layer "B.Cu") (net 27))
+  (segment (start 194.5 69.75) (end 193.3 70.95) (width 0.25) (layer "B.Cu") (net 27))
   (segment (start 196.3 90.7) (end 196.3 80.4) (width 0.25) (layer "B.Cu") (net 27))
   (segment (start 194.5 74) (end 194.5 80.1) (width 0.25) (layer "B.Cu") (net 27))
@@
   (segment (start 186.725 72.775) (end 185.24 74.26) (width 0.25) (layer "B.Cu") (net 27))
   (segment (start 118.51 71.74) (end 116.5 73.75) (width 0.25) (layer "B.Cu") (net 27))
+  (segment (start 188.55 70.95) (end 185.24 74.26) (width 0.25) (layer "B.Cu") (net 27))
   (segment (start 193.275 72.775) (end 186.725 72.775) (width 0.25) (layer "B.Cu") (net 27))
   (segment (start 193.05 98.086396) (end 192.436396 98.7) (width 0.25) (layer "B.Cu") (net 27))
